Commit message: scanning added

File: urdf/quadrotor_hokuyo_utm30lx.gazebo.xacro (robot description, xacro)
@@ -1,5 +1,5 @@
 <?xml version="1.0"?>
 <robot name="quadrotor" xmlns:xacro="http://ros.org/wiki/xacro">
-    <xacro:include filename="$(find hector_quadrotor_description)/urdf/quadrotor_hokuyo_utm30lx.urdf.xacro" />
+    <xacro:include filename="$(find uav_practice161129)/urdf/quadrotor_hokuyo_utm30lx.urdf.xacro" />
     <xacro:include filename="$(find hector_quadrotor_gazebo)/urdf/quadrotor_plugins.gazebo.xacro" />
 </robot>

File: urdf/quadrotor_hokuyo_utm30lx.urdf.xacro (robot description, xacro)
@@ -15,5 +15,5 @@
     </xacro:hokuyo_utm30lx>
     <xacro:hokuyo_utm30lx name="laser1" parent="base_link" ros_topic="scan" update_rate="40" ray_count="1081" min_angle="-135" max_angle="135">
-      <origin xyz="0.0 0.0 -0.05" rpy="${M_PI/2} 0 0"/>
+      <origin xyz="0.0 0.0 -0.07" rpy="${M_PI/2} ${M_PI/2} 0"/>
     </xacro:hokuyo_utm30lx>
     <!-- Forward facing camera -->
