Commit message: additional updates for subsumption

File: urdf/quadrotor_hokuyo_utm30lx.urdf.xacro (robot description, xacro)
@@ -11,9 +11,12 @@
     <!-- Hokuyo UTM-30LX mounted upside down below the quadrotor body -->
     <xacro:include filename="$(find hector_sensors_description)/urdf/hokuyo_utm30lx.urdf.xacro" />
-    <xacro:hokuyo_utm30lx name="laser0" parent="base_link" ros_topic="scan" update_rate="40" ray_count="1081" min_angle="-135" max_angle="135">
+    <xacro:hokuyo_utm30lx name="laser_h" parent="base_link" ros_topic="scan" update_rate="40" ray_count="1081" min_angle="-135" max_angle="135">
       <origin xyz="0.0 0.0 0.097" rpy="0 0 0"/>
     </xacro:hokuyo_utm30lx>
-    <xacro:hokuyo_utm30lx name="laser1" parent="base_link" ros_topic="scan" update_rate="40" ray_count="1081" min_angle="-135" max_angle="135">
-      <origin xyz="0.0 0.0 -0.07" rpy="${M_PI/2} ${M_PI/2} 0"/>
+    <xacro:hokuyo_utm30lx name="laser_d" parent="base_link" ros_topic="scan" update_rate="40" ray_count="1081" min_angle="-135" max_angle="135">
+      <origin xyz="0.0 0.0 -0.07" rpy="${-M_PI/2} ${M_PI/2} 0"/>
+    </xacro:hokuyo_utm30lx>
+    <xacro:hokuyo_utm30lx name="laser_u" parent="base_link" ros_topic="scan" update_rate="40" ray_count="1081" min_angle="-135" max_angle="135">
+      <origin xyz="0.0 0.0 0.160" rpy="${-M_PI/2} ${-M_PI/2} 0"/>
     </xacro:hokuyo_utm30lx>
     <!-- Forward facing camera -->
