Commit message: Clean urdf files

File: urdf/quadrotor_ray_sensor.urdf.xacro (robot description, xacro)
@@ -82,8 +82,8 @@
     </xacro:hokuyo_utm30lx>
     -->
-    <!-- Forward facing camera -->
+    <!-- Forward facing camera
     <xacro:include filename="$(find hector_sensors_description)/urdf/generic_camera.urdf.xacro" />
     <xacro:generic_camera name="front_cam" parent="base_link" ros_topic="camera/image" cam_info_topic="camera/camera_info" update_rate="10" res_x="320" res_y="240" image_format="R8G8B8" hfov="90">
       <origin xyz="0.05 0.0 -0.06" rpy="0 0 0"/>
-    </xacro:generic_camera>
+    </xacro:generic_camera> -->
 </robot>

File: urdf/quadrotor_simple.urdf.xacro (robot description, xacro)
@@ -1,6 +1,4 @@
 <?xml version="1.0"?>
 <robot xmlns:xacro="http://ros.org/wiki/xacro">
-  <xacro:include filename="$(find hector_sensors_description)/urdf/sonar_sensor.urdf.xacro" />
-  <xacro:property name="pi" value="3.1415926535897931" />
   <!-- Main quadrotor link -->
   <xacro:macro name="quadrotor_base_macro">

Commit message: Add arguments for ranging sensor in xacro

File: urdf/quadrotor_ray_sensor.urdf.xacro (robot description, xacro)
@@ -4,4 +4,7 @@
   xmlns:xacro="http://www.ros.org/wiki/xacro"
 >
+    <xacro:arg name="rate" default="20"/>
+    <xacro:arg name="min_range" default="0.01"/>
+    <xacro:arg name="max_range" default="10.0"/>
     <xacro:property name="M_PI" value="3.1415926535897931" />
     <!-- Included URDF Files -->
@@ -12,7 +15,7 @@
     <!-- ray sensors -->
     <xacro:include filename="$(find hector_sensors_description)/urdf/sonar_sensor.urdf.xacro" />
-    <xacro:property name="RATE" value="20" />
-    <xacro:property name="MIN" value="0.01" />
-    <xacro:property name="MAX" value="10.0" />
+    <xacro:property name="RATE" value="$(arg rate)" />
+    <xacro:property name="MIN" value="$(arg min_range)" />
+    <xacro:property name="MAX" value="$(arg max_range)" />
     <xacro:property name="DEG" value="3" />
     <xacro:property name="STEP_X" value="0.05" />
