Commit message: Make all gazebo.xacro files accept parameters

File: urdf/adhoc/quadrotor_adhoc.gazebo.xacro (robot description, xacro)
@@ -1,6 +1,26 @@
 <?xml version="1.0"?>
 <robot name="quadrotor" xmlns:xacro="http://ros.org/wiki/xacro">
+    <xacro:arg name="disable_imu" default="false"/>
+    <xacro:arg name="disable_baro" default="false"/>
+    <xacro:arg name="disable_magnetic" default="false"/>
+    <xacro:arg name="disable_gps" default="false"/>
+    <xacro:arg name="disable_groundtruth" default="false"/>
     <xacro:include filename="$(find quadrotor_tunnel_nav)/urdf/quadrotor_ray_sensor.urdf.xacro" />
-    <xacro:include filename="$(find quadrotor_tunnel_nav)/urdf/quadrotor_plugins_cusom.gazebo.xacro" />
+    <xacro:include filename="$(find quadrotor_tunnel_nav)/urdf/plugins.gazebo.xacro" />
+    <xacro:unless value="$(arg disable_imu)">
+      <xacro:quadrotor_imu />
+    </xacro:unless>
+    <xacro:unless value="$(arg disable_baro)">
+      <xacro:quadrotor_baro />
+    </xacro:unless>
+    <xacro:unless value="$(arg disable_magnetic)">
+      <xacro:quadrotor_magnetic />
+    </xacro:unless>
+    <xacro:unless value="$(arg disable_gps)">
+      <xacro:quadrotor_gps />
+    </xacro:unless>
+    <xacro:unless value="$(arg disable_groundtruth)">
+      <xacro:quadrotor_groundtruth />
+    </xacro:unless>
     <gazebo>
       <plugin name="adhocclient_plugin" filename="libAdHocClientPlugin.so">

File: urdf/plugins.gazebo.xacro (robot description, xacro)
@@ -1,6 +1,15 @@
 <?xml version="1.0"?>
 <robot xmlns:xacro="http://www.ros.org/wiki/xacro">
+  <xacro:arg name="world_frame" default="world"/>
+  <xacro:arg name="base_link_frame" default="base_link"/>
+  <xacro:include filename="$(find hector_quadrotor_gazebo)/urdf/quadrotor_controller.gazebo.xacro" />
+  <xacro:include filename="$(find hector_quadrotor_gazebo)/urdf/quadrotor_propulsion.gazebo.xacro" />
+  <xacro:include filename="$(find hector_quadrotor_gazebo)/urdf/quadrotor_aerodynamics.gazebo.xacro" />
+  <!-- Quadrotor Gazebo Plugins -->
+  <xacro:quadrotor_controller />
+  <xacro:quadrotor_propulsion />
+  <xacro:quadrotor_aerodynamics />
   <!-- Quadrotor Sensor Plugins -->
-  <xacro:macro name="quadrotor_sensors">
+  <xacro:macro name="quadrotor_imu">
         <gazebo>
           <plugin name="quadrotor_imu_sim" filename="libhector_gazebo_ros_imu.so">
@@ -16,4 +25,8 @@
             <rateGaussianNoise>0.05 0.05 0.015</rateGaussianNoise>
           </plugin>
+        </gazebo>
+  </xacro:macro>
+  <xacro:macro name="quadrotor_baro">
+        <gazebo>
           <plugin name="quadrotor_baro_sim" filename="libhector_gazebo_ros_baro.so">
             <updateRate>10.0</updateRate>
@@ -26,4 +39,8 @@
             <gaussianNoise>0.1</gaussianNoise>
           </plugin>
+        </gazebo>
+  </xacro:macro>
+  <xacro:macro name="quadrotor_magnetic">
+        <gazebo>
           <plugin name="quadrotor_magnetic_sim" filename="libhector_gazebo_ros_magnetic.so">
             <updateRate>10.0</updateRate>
@@ -35,4 +52,8 @@
             <gaussianNoise>1.3e-2 1.3e-2 1.3e-2</gaussianNoise>
           </plugin>
+        </gazebo>
+  </xacro:macro>
+  <xacro:macro name="quadrotor_gps">
+        <gazebo>
           <plugin name="quadrotor_gps_sim" filename="libhector_gazebo_ros_gps.so">
             <updateRate>4.0</updateRate>
@@ -48,4 +69,8 @@
             <velocityGaussianNoise>0.05 0.05 0.05</velocityGaussianNoise>
           </plugin>
+        </gazebo>
+  </xacro:macro>
+  <xacro:macro name="quadrotor_groundtruth">
+        <gazebo>
           <plugin name="quadrotor_groundtruth_sim" filename="libgazebo_ros_p3d.so">
             <updateRate>100.0</updateRate>

File: urdf/quadrotor_ray_sensor.gazebo.xacro (robot description, xacro)
@@ -1,5 +1,25 @@
 <?xml version="1.0"?>
 <robot name="quadrotor" xmlns:xacro="http://www.ros.org/wiki/xacro">
+    <xacro:arg name="disable_imu" default="false"/>
+    <xacro:arg name="disable_baro" default="false"/>
+    <xacro:arg name="disable_magnetic" default="false"/>
+    <xacro:arg name="disable_gps" default="false"/>
+    <xacro:arg name="disable_groundtruth" default="false"/>
     <xacro:include filename="$(find quadrotor_tunnel_nav)/urdf/quadrotor_ray_sensor.urdf.xacro" />
-    <xacro:include filename="$(find quadrotor_tunnel_nav)/urdf/quadrotor_plugins_custom.gazebo.xacro" />
+    <xacro:include filename="$(find quadrotor_tunnel_nav)/urdf/plugins.gazebo.xacro" />
+    <xacro:unless value="$(arg disable_imu)">
+      <xacro:quadrotor_imu />
+    </xacro:unless>
+    <xacro:unless value="$(arg disable_baro)">
+      <xacro:quadrotor_baro />
+    </xacro:unless>
+    <xacro:unless value="$(arg disable_magnetic)">
+      <xacro:quadrotor_magnetic />
+    </xacro:unless>
+    <xacro:unless value="$(arg disable_gps)">
+      <xacro:quadrotor_gps />
+    </xacro:unless>
+    <xacro:unless value="$(arg disable_groundtruth)">
+      <xacro:quadrotor_groundtruth />
+    </xacro:unless>
 </robot>

File: urdf/quadrotor_ray_sensor.urdf.xacro (robot description, xacro)
@@ -9,5 +9,5 @@
     <xacro:property name="M_PI" value="3.1415926535897931" />
     <!-- Included URDF Files -->
-    <xacro:include filename="$(find quadrotor_tunnel_nav)/urdf/quadrotor_simple.urdf.xacro" />
+    <xacro:include filename="$(find quadrotor_tunnel_nav)/urdf/quadrotor_base.urdf.xacro" />
     <!-- Instantiate quadrotor_base_macro once (has no parameters atm) -->
     <!-- page: http://wiki.ros.org/hector_gazebo_plugins#GazeboRosSonar -->
